Commit message: Sync ZX200 joint origins with zx200_ros2 URDF
zx200_ros2 main moved the working-range joint origins (PR #21, commit
3503f1b), so the ZX200 model in MainScene has to follow.

Assets/Scenes/MainScene.unity - the three link transforms in the zx200
hierarchy (Unity frame, y and z swapped against the URDF):
  boom_link    (0.040187, 0.83669, 0.22767) -> (0.040187, 0.72492, 0.05467)
  arm_link     (-0.010957, 2.9959, 4.7878)  -> (-0.010957, 3.00227, 4.83998)
  bucket_link  (0.023546, 2.1809, 1.8954)   -> (0.023546, 2.17374, 1.91546)

and the matching connected frames of the constraints that define those
joints, which live in the parent link frame and therefore carry the joint
origin as well:
  AGXUnity.Hinge_boom_body  (parent body_link)
  AGXUnity.Hinge_arm_boom   (parent boom_link)
  AGXUnity.Hinge_bucket_arm (parent arm_link)

Only translations change. The joint axis orientations are unaffected because
the URDF origin rotations (32.0357/16.9707/-9.20083 deg) did not change;
the cylinder attachment frames (boom/arm/bucket tilt cylinders, H/I links,
rods) are expressed relative to the link frames they are attached to and
stay valid.

Assets/Machines/Excavator/zx200/zx200.urdf is the URDF the model numbers
were taken from and still had the old origins; it is updated to the same
values so both agree.

Checked by re-parsing the scene: in the zx200 subtree the three link
transforms and the connected frames of the three hinges all read the new
origins, and no occurrence of the old origins is left in the model.

File: Assets/Machines/Excavator/zx200/zx200.urdf (robot description, URDF)
Before this commit: robot zx200, 14 links, 13 joints
Joints:
- joint joint2: origin xyz=0.22767 -0.040187 0.83669 -> xyz=0.05467 -0.040187 0.72492
- joint joint3: origin xyz=4.7878 0.010957 2.9959 -> xyz=4.83998 0.010957 3.00227
- joint joint4: origin xyz=1.8954 -0.023546 2.1809 -> xyz=1.91546 -0.023546 2.17374

Commit message: Align ZX200 hinge zeros with the URDF joint-origin rotations
Only the joint origins (translations) were synced so far; the joint zeros of the
AGX model were still the ones the scene happened to be saved in, so the angles
exchanged with MoveIt over the Unity bridge would have carried a constant offset
of the difference in rpy.

How the AGX zero is defined in this model:
  * each hinge (AGXUnity.Hinge_<child>_<parent>) holds a reference frame on the
    child link (R_ref) and a connected frame on the parent link (R_con); the
    hinge angle is measured about the frames' common z axis and is zero when the
    two frames are aligned, i.e. at phi = R_con * R_ref^-1 (child relative to
    parent);
  * the scenes were authored with m_synchronized = 1, and
    AGXUnity.AttachmentPair.Synchronize() - called from Constraint.Initialize -
    overwrites the connected frame with the reference frame. The zero was
    therefore simply "the pose the scene was saved in" (measurably
    +21.35 / +61.68 / -16.25 deg for boom/arm/bucket), which is also why the
    serialized frames exactly coincide at the saved pose.

Change: turn the synchronization off so the authored frames define the zero, and
rotate the connected frame by the twist that moves the zero onto the URDF rpy
(Rx(rpy) in Unity terms, i.e. the URDF's rotation about +y):

  boom_body   +21.35   -> +32.0357  deg   (twist +10.6857  deg about the frame z)
  arm_boom    +61.68   -> +16.9707  deg   (twist +44.7093  deg)
  bucket_arm  -16.25   -> -9.20083  deg   (twist  +7.0492  deg)

Only the rotation of the connected frame is touched, so the joint origins and the
hinge axis are unchanged (verified: the correction is a pure twist about the
frame's local z, the frame's z axis in the parent link drifts by < 1e-7, and
R_con * R_ref^-1 comes out as exactly Rx(rpy) afterwards). The hinge has no angle
range serialized (the RR row is disabled with range (-inf, inf)), so no limits
have to be shifted.

The zx200 link poses in the scene are not touched. With the zero now fixed, the
machine's saved pose reads as its real URDF joint angles instead of (0, 0, 0):
about -10.69 deg (boom), +44.71 deg (arm), -7.05 deg (bucket); the swing joint
already had the correct zero (0). Note the auxiliary linkage links keep their own
frames, so if the machine ever needs to start at the URDF zero pose the scene
pose has to be re-authored (and its closed chain re-solved), not just these
frames.

Assets/Machines/Excavator/zx200/zx200.urdf, the model's source document, had no
rpy on joints 2/3/4 at all; it now carries the same rotations as zx200_ros2.

File: Assets/Machines/Excavator/zx200/zx200.urdf (robot description, URDF)
Before this commit: robot zx200, 14 links, 13 joints
Joints:
- joint joint2: origin xyz=0.05467 -0.040187 0.72492 -> xyz=0.05467 -0.040187 0.72492 rpy=0 0.5591284432 0
- joint joint3: origin xyz=4.83998 0.010957 3.00227 -> xyz=4.83998 0.010957 3.00227 rpy=0 0.2961945914 0
- joint joint4: origin xyz=1.91546 -0.023546 2.17374 -> xyz=1.91546 -0.023546 2.17374 rpy=0 -0.1605847774 0
